File: kicad/top_level/top_level.kicad_sch (KiCad schematic)
At the start: 0 parts

Commit message: files
Other:
- added sheet INSTRUCTION DECODE (decode\id.kicad_sch)
- added sheet PROCESSOR STATUS REGISTER (registers\p.kicad_sch)
- added sheet PROGRAM COUNTER HIGH (pc\pc.kicad_sch)
- added sheet PROGRAM COUNTER LOW (pc\pc.kicad_sch)
Changed lines of the file:
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@@
+    )
+  )
+  (sheet (at 237.49 133.35) (size 19.05 17.78) (fields_autoplaced)
+    (stroke (width 0.1524) (type solid) (color 0 0 0 0))
+    (fill (color 0 0 0 0.0000))
+    (property "Sheet name" "PROGRAM COUNTER HIGH" (id 0) (at 237.49 132.6384 0)
+      (effects (font (size 1.27 1.27)) (justify left bottom))
+    )
+    (property "Sheet file" "pc\\pc.kicad_sch" (id 1) (at 237.49 151.7146 0)
+      (effects (font (size 1.27 1.27)) (justify left top))
     )
   )
@@
     )
   )
+  (sheet (at 210.82 133.35) (size 19.05 17.78) (fields_autoplaced)
+    (stroke (width 0.1524) (type solid) (color 0 0 0 0))
+    (fill (color 0 0 0 0.0000))
+    (property "Sheet name" "PROGRAM COUNTER LOW" (id 0) (at 210.82 132.6384 0)
+      (effects (font (size 1.27 1.27)) (justify left bottom))
+    )
+    (property "Sheet file" "pc\\pc.kicad_sch" (id 1) (at 210.82 151.7146 0)
+      (effects (font (size 1.27 1.27)) (justify left top))
+    )
+  )
   (sheet (at 182.88 110.49) (size 12.7 11.43) (fields_autoplaced)
     (stroke (width 0.1524) (type solid) (color 0 0 0 0))
@@
     )
     (property "Sheet file" "registers\\reg_siso.kicad_sch" (id 1) (at 105.41 109.8046 0)
+      (effects (font (size 1.27 1.27)) (justify left top))
+    )
+  )
+  (sheet (at 209.55 99.06) (size 24.13 20.32) (fields_autoplaced)
+    (stroke (width 0.1524) (type solid) (color 0 0 0 0))
+    (fill (color 0 0 0 0.0000))
+    (property "Sheet name" "PROCESSOR STATUS REGISTER" (id 0) (at 209.55 98.3484 0)
+      (effects (font (size 1.27 1.27)) (justify left bottom))
+    )
+    (property "Sheet file" "registers\\p.kicad_sch" (id 1) (at 209.55 119.9646 0)
+      (effects (font (size 1.27 1.27)) (justify left top))
+    )
+  )
+  (sheet (at 179.07 133.35) (size 16.51 15.24) (fields_autoplaced)
+    (stroke (width 0.1524) (type solid) (color 0 0 0 0))
+    (fill (color 0 0 0 0.0000))
+    (property "Sheet name" "INSTRUCTION DECODE" (id 0) (at 179.07 132.6384 0)
+      (effects (font (size 1.27 1.27)) (justify left bottom))
+    )
+    (property "Sheet file" "decode\\id.kicad_sch" (id 1) (at 179.07 149.1746 0)
       (effects (font (size 1.27 1.27)) (justify left top))
     )
@@
     (path "/f5cf2763-2c3c-47b5-9c94-b5631851b114/8a47721d-ec29-4274-8fda-1028caa4df53" (page "10"))
     (path "/f5cf2763-2c3c-47b5-9c94-b5631851b114" (page "11"))
+    (path "/48a6da7e-9214-438f-b562-3df14a9a3c45" (page "12"))
     (path "/cf533c45-c632-483f-ae69-36538f7b8a37" (page "14"))
+    (path "/f4c1987e-1abd-4604-acec-54db97a4dd27" (page "15"))
+    (path "/97f7bdfb-063c-422d-933c-6d8278ccd0d3" (page "16"))
+    (path "/e1f48394-fb09-4abd-a461-39038b654295" (page "18"))
     (path "/dcf4f85a-aa88-4be5-970a-6e101386f216/8a47721d-ec29-4274-8fda-1028caa4df53" (page ""))
     (path "/dcf4f85a-aa88-4be5-970a-6e101386f216" (page "#"))

Commit message: try to fix paths
Other:
- added sheet A INPUT (registers/reg_diso.kicad_sch)
- added sheet ACCUMULATOR (registers/reg_sido.kicad_sch)
- added sheet ADDER HOLD REGISTER (registers/reg_sido.kicad_sch)
- added sheet B INPUT (registers\reg_tiso.kicad_sch)
- added sheet INPUT DATA LATCH (registers/reg_sito.kicad_sch)
- added sheet STACK POINTER (registers/reg_sido.kicad_sch)
- sheet ADDRESS HIGH REGISTER: file registers\reg_siso.kicad_sch -> registers/reg_siso.kicad_sch
- sheet ADDRESS LOW REGISTER: file registers\reg_siso.kicad_sch -> registers/reg_siso.kicad_sch
- sheet ALU: file alu\alu.kicad_sch -> alu/alu.kicad_sch
- sheet DATA OUTPUT REGISTER: file registers\reg_siso.kicad_sch -> registers/reg_siso.kicad_sch
- sheet INSTRUCTION DECODE: file decode\id.kicad_sch -> decode/id.kicad_sch
- sheet INSTRUCTION REGISTER: file registers\reg_siso.kicad_sch -> registers/reg_siso.kicad_sch
- sheet PROCESSOR STATUS REGISTER: file registers\p.kicad_sch -> registers/p.kicad_sch
- sheet PROGRAM COUNTER HIGH: file pc\pc.kicad_sch -> pc/pc.kicad_sch
- sheet PROGRAM COUNTER LOW: file pc\pc.kicad_sch -> pc/pc.kicad_sch
- sheet X INDEX REGISTER: file registers\reg_siso.kicad_sch -> registers/reg_siso.kicad_sch
- sheet Y INDEX REGISTER1: file registers\reg_siso.kicad_sch -> registers/reg_siso.kicad_sch
