File: kicad/top_level/registers/reg_diso.kicad_sch (KiCad schematic)
At the start: 1 part

Commit message: try to fix paths
Parts:
- removed U?: 74AHC244, symbol 74xx:74AHC244
- added U?: 74AHC244, symbol 74xx:74AHC244
Connections:
- net +5V: now also U?.20 (VCC)
- net GND: now also U?.10 (GND)
- net bus_enable: now also U?.1 (1OE), U?.19 (2OE)
- net d0: now also U?.18 (1Y0)
- net d1: now also U?.16 (1Y1)
- net d2: now also U?.14 (1Y2)
- net d3: now also U?.12 (1Y3)
- net d4: now also U?.3 (2Y0)
- net d5: now also U?.5 (2Y1)
- net d6: now also U?.7 (2Y2)
- net d7: now also U?.9 (2Y3)
- net regled/q0: now also U?.2 (1A0)
- net regled/q1: now also U?.4 (1A1)
- net regled/q2: now also U?.6 (1A2)
- net regled/q3: now also U?.8 (1A3)
- net regled/q4: now also U?.17 (2A0)
- net regled/q5: now also U?.15 (2A1)
- net regled/q6: now also U?.13 (2A2)
- net regled/q7: now also U?.11 (2A3)
Changed lines of the file:
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@@
     (effects (font (size 1.27 1.27)) (justify right))
   )
-  (symbol (lib_id "74xx:74AHC244") (at 172.72 91.44 0)
+  (symbol (lib_id "power:GND") (at 172.72 111.76 0) (unit 1)
+    (in_bom yes) (on_board yes) (fields_autoplaced)
+    (property "Reference" "#PWR?" (id 0) (at 172.72 118.11 0)
+      (effects (font (size 1.27 1.27)) hide)
+    )
+    (property "Value" "GND" (id 1) (at 172.72 116.84 0))
+    (property "Footprint" "" (id 2) (at 172.72 111.76 0)
+      (effects (font (size 1.27 1.27)) hide)
+    )
+    (property "Datasheet" "" (id 3) (at 172.72 111.76 0)
+      (effects (font (size 1.27 1.27)) hide)
+    )
+    (pin "1")
+  )
+  (symbol (lib_id "power:+5V") (at 172.72 71.12 0) (unit 1)
+    (in_bom yes) (on_board yes) (fields_autoplaced)
+    (property "Reference" "#PWR?" (id 0) (at 172.72 74.93 0)
+      (effects (font (size 1.27 1.27)) hide)
+    )
+    (property "Value" "+5V" (id 1) (at 172.72 66.04 0))
+    (property "Footprint" "" (id 2) (at 172.72 71.12 0)
+      (effects (font (size 1.27 1.27)) hide)
+    )
+    (property "Datasheet" "" (id 3) (at 172.72 71.12 0)
+      (effects (font (size 1.27 1.27)) hide)
+    )
+    (pin "1")
+  )
+  (symbol (lib_id "74xx:74AHC244") (at 172.72 91.44 0) (unit 1)
     (in_bom yes) (on_board yes) (fields_autoplaced)
     (property "Reference" "U?" (id 0) (at 174.7394 71.12 0)
@@
     (pin "9")
   )
-  (symbol (lib_id "power:GND") (at 172.72 111.76 0)
-    (in_bom yes) (on_board yes) (fields_autoplaced)
-    (property "Reference" "#PWR?" (id 0) (at 172.72 118.11 0)
-      (effects (font (size 1.27 1.27)) hide)
-    )
-    (property "Value" "GND" (id 1) (at 172.72 116.84 0))
-    (property "Footprint" "" (id 2) (at 172.72 111.76 0)
-      (effects (font (size 1.27 1.27)) hide)
-    )
-    (property "Datasheet" "" (id 3) (at 172.72 111.76 0)
-      (effects (font (size 1.27 1.27)) hide)
-    )
-    (pin "1")
-  )
-  (symbol (lib_id "power:+5V") (at 172.72 71.12 0)
-    (in_bom yes) (on_board yes) (fields_autoplaced)
-    (property "Reference" "#PWR?" (id 0) (at 172.72 74.93 0)
-      (effects (font (size 1.27 1.27)) hide)
-    )
-    (property "Value" "+5V" (id 1) (at 172.72 66.04 0))
-    (property "Footprint" "" (id 2) (at 172.72 71.12 0)
-      (effects (font (size 1.27 1.27)) hide)
-    )
-    (property "Datasheet" "" (id 3) (at 172.72 71.12 0)
-      (effects (font (size 1.27 1.27)) hide)
-    )
-    (pin "1")
-  )
   (sheet (at 132.08 76.2) (size 17.78 26.67) (fields_autoplaced)
